Commit message: Changed project name to mini_car in every file

File: urdf/my_robot_integration.urdf.xacro (robot description, xacro)
@@ -5,6 +5,6 @@
 	<!-- Include Robot's urdf filepath -->
 	<!-- Include Lidar's urdf filepath -->
-	<xacro:include filename="/home/ameya/catkin_ws/src/enpm662_proj1_urdf/urdf/enpm662_proj1_urdf.urdf"/>
-	<xacro:include filename="/home/ameya/catkin_ws/src/enpm662_proj1_urdf/urdf/ydlidar.urdf"/>
+	<xacro:include filename="/home/ninadharish/catkin_ws/src/enpm662_proj1_urdf/urdf/enpm662_proj1_urdf.urdf"/>
+	<xacro:include filename="/home/ninadharish/catkin_ws/src/enpm662_proj1_urdf/urdf/ydlidar.urdf"/>
 <!-- Add your gazebo sensors here -->
 <gazebo reference="base_laser">

File: urdf/project1_integrated.urdf (robot description, URDF)
Before this commit: robot mini_car, 9 links, 8 joints
Links:
- link base_laser: geometry collision mesh filename=package://mini_car/meshes/ydlidar.dae; visual mesh filename=package://mini_car/meshes/ydlidar.dae
- link chassis: geometry collision mesh filename=package://mini_car/meshes/chassis.STL; visual mesh filename=package://mini_car/meshes/chassis.STL
- link left_front_steer: geometry collision mesh filename=package://mini_car/meshes/left_front_steer.STL; visual mesh filename=package://mini_car/meshes/left_front_steer.STL
- link left_wheel: geometry collision mesh filename=package://mini_car/meshes/left_wheel.STL; visual mesh filename=package://mini_car/meshes/left_wheel.STL
- link rear_drive: geometry collision mesh filename=package://mini_car/meshes/rear_drive.STL; visual mesh filename=package://mini_car/meshes/rear_drive.STL
- link right_front_steer: geometry collision mesh filename=package://mini_car/meshes/right_front_steer.STL; visual mesh filename=package://mini_car/meshes/right_front_steer.STL
- link right_wheel: geometry collision mesh filename=package://mini_car/meshes/right_wheel.STL; visual mesh filename=package://mini_car/meshes/right_wheel.STL
Joints:
- joint left_front_steer_joint: limit lower=0 upper=0 effort=0 velocity=0 -> lower=0 upper=0 effort=10 velocity=50
- joint left_wheel_joint: limit lower=0 upper=0 effort=0 velocity=0 -> lower=0 upper=0 effort=10 velocity=50
- joint rear_drive_joint: limit lower=0 upper=0 effort=0 velocity=0 -> lower=0 upper=0 effort=10 velocity=50
- joint right_front_steer_joint: limit lower=0 upper=0 effort=0 velocity=0 -> lower=0 upper=0 effort=10 velocity=50
- joint right_wheel_joint: limit lower=0 upper=0 effort=0 velocity=0 -> lower=0 upper=0 effort=10 velocity=50
